File: pcb/yosino46.sch (KiCad schematic (older format))
At the start: 85 parts, among them J0 LED, J1 TRRS, J2 OLED, J3 OLED, J4 OLED, SW1 SW_PUSH, SW10 SW_PUSH, SW11 SW_PUSH, SW12 SW_PUSH, SW13 SW_PUSH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

Commit message: yosino46作成
Parts:
- removed J2: OLED, yosino46:OLED, symbol Connector_Generic:Conn_01x04
- L1, L10, L11, L12, L13, L14, L15, L16, L17, L18, L19, L2, L20, L21, L22, L23, L3, L4, L5, L6, L7, L8, L9: footprint yosino46:SK6812MINI_rev -> yosino46:SK6812MINI_padin_rev
Changed lines of the file:
@@
 F 0 "L6" H 9675 4287 51  0000 C CNN
 F 1 "SK6812MINI" H 9675 4222 16  0000 C CNN
-F 2 "yosino46:SK6812MINI_rev" H 9675 4025 60  0001 C CNN
+F 2 "yosino46:SK6812MINI_padin_rev" H 9675 4025 60  0001 C CNN
 F 3 "" H 9675 4025 60  0001 C CNN
 	1    9675 4025
@@
 F 0 "L5" H 9175 4287 51  0000 C CNN
 F 1 "SK6812MINI" H 9175 4222 16  0000 C CNN
-F 2 "yosino46:SK6812MINI_rev" H 9175 4025 60  0001 C CNN
+F 2 "yosino46:SK6812MINI_padin_rev" H 9175 4025 60  0001 C CNN
 F 3 "" H 9175 4025 60  0001 C CNN
 	1    9175 4025
@@
 F 0 "L4" H 8675 4287 51  0000 C CNN
 F 1 "SK6812MINI" H 8675 4222 16  0000 C CNN
-F 2 "yosino46:SK6812MINI_rev" H 8675 4025 60  0001 C CNN
+F 2 "yosino46:SK6812MINI_padin_rev" H 8675 4025 60  0001 C CNN
 F 3 "" H 8675 4025 60  0001 C CNN
 	1    8675 4025
@@
 F 0 "L3" H 8175 4287 51  0000 C CNN
 F 1 "SK6812MINI" H 8175 4222 16  0000 C CNN
-F 2 "yosino46:SK6812MINI_rev" H 8175 4025 60  0001 C CNN
+F 2 "yosino46:SK6812MINI_padin_rev" H 8175 4025 60  0001 C CNN
 F 3 "" H 8175 4025 60  0001 C CNN
 	1    8175 4025
@@
 F 0 "L2" H 7675 4287 51  0000 C CNN
 F 1 "SK6812MINI" H 7675 4222 16  0000 C CNN
-F 2 "yosino46:SK6812MINI_rev" H 7675 4025 60  0001 C CNN
+F 2 "yosino46:SK6812MINI_padin_rev" H 7675 4025 60  0001 C CNN
 F 3 "" H 7675 4025 60  0001 C CNN
 	1    7675 4025
@@
 F 0 "L1" H 7175 4287 51  0000 C CNN
 F 1 "SK6812MINI" H 7175 4222 16  0000 C CNN
-F 2 "yosino46:SK6812MINI_rev" H 7175 4025 60  0001 C CNN
+F 2 "yosino46:SK6812MINI_padin_rev" H 7175 4025 60  0001 C CNN
 F 3 "" H 7175 4025 60  0001 C CNN
 	1    7175 4025
@@
 F 0 "L7" H 7175 4313 51  0000 C CNN
 F 1 "SK6812MINI" H 7175 4378 16  0000 C CNN
-F 2 "yosino46:SK6812MINI_rev" H 7175 4575 60  0001 C CNN
+F 2 "yosino46:SK6812MINI_padin_rev" H 7175 4575 60  0001 C CNN
 F 3 "" H 7175 4575 60  0001 C CNN
 	1    7175 4575
@@
 F 0 "L8" H 7675 4313 51  0000 C CNN
 F 1 "SK6812MINI" H 7675 4378 16  0000 C CNN
-F 2 "yosino46:SK6812MINI_rev" H 7675 4575 60  0001 C CNN
+F 2 "yosino46:SK6812MINI_padin_rev" H 7675 4575 60  0001 C CNN
 F 3 "" H 7675 4575 60  0001 C CNN
 	1    7675 4575
@@
 F 0 "L9" H 8175 4313 51  0000 C CNN
 F 1 "SK6812MINI" H 8175 4378 16  0000 C CNN
-F 2 "yosino46:SK6812MINI_rev" H 8175 4575 60  0001 C CNN
+F 2 "yosino46:SK6812MINI_padin_rev" H 8175 4575 60  0001 C CNN
 F 3 "" H 8175 4575 60  0001 C CNN
 	1    8175 4575
@@
 F 0 "L10" H 8675 4313 51  0000 C CNN
 F 1 "SK6812MINI" H 8675 4378 16  0000 C CNN
-F 2 "yosino46:SK6812MINI_rev" H 8675 4575 60  0001 C CNN
+F 2 "yosino46:SK6812MINI_padin_rev" H 8675 4575 60  0001 C CNN
 F 3 "" H 8675 4575 60  0001 C CNN
 	1    8675 4575
@@
 F 0 "L11" H 9175 4313 51  0000 C CNN
 F 1 "SK6812MINI" H 9175 4378 16  0000 C CNN
-F 2 "yosino46:SK6812MINI_rev" H 9175 4575 60  0001 C CNN
+F 2 "yosino46:SK6812MINI_padin_rev" H 9175 4575 60  0001 C CNN
 F 3 "" H 9175 4575 60  0001 C CNN
 	1    9175 4575
@@
 F 0 "L12" H 9675 4313 51  0000 C CNN
 F 1 "SK6812MINI" H 9675 4378 16  0000 C CNN
-F 2 "yosino46:SK6812MINI_rev" H 9675 4575 60  0001 C CNN
+F 2 "yosino46:SK6812MINI_padin_rev" H 9675 4575 60  0001 C CNN
 F 3 "" H 9675 4575 60  0001 C CNN
 	1    9675 4575
@@
 F 0 "L18" H 9675 5387 51  0000 C CNN
 F 1 "SK6812MINI" H 9675 5322 16  0000 C CNN
-F 2 "yosino46:SK6812MINI_rev" H 9675 5125 60  0001 C CNN
+F 2 "yosino46:SK6812MINI_padin_rev" H 9675 5125 60  0001 C CNN
 F 3 "" H 9675 5125 60  0001 C CNN
 	1    9675 5125
@@
 F 0 "L17" H 9175 5387 51  0000 C CNN
 F 1 "SK6812MINI" H 9175 5322 16  0000 C CNN
-F 2 "yosino46:SK6812MINI_rev" H 9175 5125 60  0001 C CNN
+F 2 "yosino46:SK6812MINI_padin_rev" H 9175 5125 60  0001 C CNN
 F 3 "" H 9175 5125 60  0001 C CNN
 	1    9175 5125
@@
 F 0 "L16" H 8675 5387 51  0000 C CNN
 F 1 "SK6812MINI" H 8675 5322 16  0000 C CNN
-F 2 "yosino46:SK6812MINI_rev" H 8675 5125 60  0001 C CNN
+F 2 "yosino46:SK6812MINI_padin_rev" H 8675 5125 60  0001 C CNN
 F 3 "" H 8675 5125 60  0001 C CNN
 	1    8675 5125
@@
 F 0 "L15" H 8175 5387 51  0000 C CNN
 F 1 "SK6812MINI" H 8175 5322 16  0000 C CNN
-F 2 "yosino46:SK6812MINI_rev" H 8175 5125 60  0001 C CNN
+F 2 "yosino46:SK6812MINI_padin_rev" H 8175 5125 60  0001 C CNN
 F 3 "" H 8175 5125 60  0001 C CNN
 	1    8175 5125
@@
 F 0 "L14" H 7675 5387 51  0000 C CNN
 F 1 "SK6812MINI" H 7675 5322 16  0000 C CNN
-F 2 "yosino46:SK6812MINI_rev" H 7675 5125 60  0001 C CNN
+F 2 "yosino46:SK6812MINI_padin_rev" H 7675 5125 60  0001 C CNN
 F 3 "" H 7675 5125 60  0001 C CNN
 	1    7675 5125
@@
 F 0 "L13" H 7175 5387 51  0000 C CNN
 F 1 "SK6812MINI" H 7175 5322 16  0000 C CNN
-F 2 "yosino46:SK6812MINI_rev" H 7175 5125 60  0001 C CNN
+F 2 "yosino46:SK6812MINI_padin_rev" H 7175 5125 60  0001 C CNN
 F 3 "" H 7175 5125 60  0001 C CNN
 	1    7175 5125
@@
 F 0 "L19" H 7175 5413 51  0000 C CNN
 F 1 "SK6812MINI" H 7175 5478 16  0000 C CNN
-F 2 "yosino46:SK6812MINI_rev" H 7175 5675 60  0001 C CNN
+F 2 "yosino46:SK6812MINI_padin_rev" H 7175 5675 60  0001 C CNN
 F 3 "" H 7175 5675 60  0001 C CNN
 	1    7175 5675
@@
 F 0 "L20" H 7675 5413 51  0000 C CNN
 F 1 "SK6812MINI" H 7675 5478 16  0000 C CNN
-F 2 "yosino46:SK6812MINI_rev" H 7675 5675 60  0001 C CNN
+F 2 "yosino46:SK6812MINI_padin_rev" H 7675 5675 60  0001 C CNN
 F 3 "" H 7675 5675 60  0001 C CNN
 	1    7675 5675
@@
 F 0 "L21" H 8175 5413 51  0000 C CNN
 F 1 "SK6812MINI" H 8175 5478 16  0000 C CNN
-F 2 "yosino46:SK6812MINI_rev" H 8175 5675 60  0001 C CNN
+F 2 "yosino46:SK6812MINI_padin_rev" H 8175 5675 60  0001 C CNN
 F 3 "" H 8175 5675 60  0001 C CNN
 	1    8175 5675
@@
 F 0 "L22" H 8675 5413 51  0000 C CNN
 F 1 "SK6812MINI" H 8675 5478 16  0000 C CNN
-F 2 "yosino46:SK6812MINI_rev" H 8675 5675 60  0001 C CNN
+F 2 "yosino46:SK6812MINI_padin_rev" H 8675 5675 60  0001 C CNN
 F 3 "" H 8675 5675 60  0001 C CNN
 	1    8675 5675
@@
 F 0 "L23" H 9175 5413 51  0000 C CNN
 F 1 "SK6812MINI" H 9175 5478 16  0000 C CNN
-F 2 "yosino46:SK6812MINI_rev" H 9175 5675 60  0001 C CNN
+F 2 "yosino46:SK6812MINI_padin_rev" H 9175 5675 60  0001 C CNN
 F 3 "" H 9175 5675 60  0001 C CNN
 	1    9175 5675
@@
 	5000 3350 4900 3350
 $Comp
-L Connector_Generic:Conn_01x04 J2
-U 1 1 5C9E1696
-P 1850 4450
-F 0 "J2" H 1850 4150 50  0000 C CNN
-F 1 "OLED" H 1850 4675 50  0000 C CNN
-F 2 "yosino46:OLED" H 1850 4450 50  0001 C CNN
-F 3 "~" H 1850 4450 50  0001 C CNN
-	1    1850 4450
-	-1   0    0    1
-$EndComp
-$Comp
 L Connector_Generic:Conn_01x03 J0
 U 1 1 5CA17D54
@@
 	2450 6100 2450 6275
 Connection ~ 2450 6100
-Wire Wire Line
-	2050 4250 2450 4250
-Wire Wire Line
-	2350 4350 2050 4350
-Wire Wire Line
-	2050 4450 2250 4450
-Wire Wire Line
-	2150 4550 2050 4550
 Connection ~ 2150 5950
 Wire Wire Line
 	2050 4875 2450 4875
-Connection ~ 2450 4875
 Wire Wire Line
 	2050 4975 2350 4975
-Connection ~ 2350 4975
 Wire Wire Line
 	2050 5075 2250 5075
-Connection ~ 2250 5075
 Wire Wire Line
 	2050 5175 2150 5175
-Connection ~ 2150 5175
 Wire Wire Line
 	3025 2400 3525 2400
@@
 $EndComp
 Wire Wire Line
-	2450 4250 2450 4875
-Wire Wire Line
 	2450 4875 2450 5500
 Wire Wire Line
-	2350 4350 2350 4975
-Wire Wire Line
-	2250 4450 2250 5075
-Wire Wire Line
-	2150 4550 2150 5175
-Wire Wire Line
 	2150 5175 2150 5800

Commit message: yosino46作成
Parts:
- L1, L10, L11, L12, L13, L14, L15, L16, L17, L18, L19, L2, L20, L21, L22, L23, L3, L4, L5, L6, L7, L8, L9: footprint yosino46:SK6812MINI_padin_rev -> yosino46:SK6812MINI_rev
Changed lines of the file:
@@
 F 0 "L6" H 9675 4287 51  0000 C CNN
 F 1 "SK6812MINI" H 9675 4222 16  0000 C CNN
-F 2 "yosino46:SK6812MINI_padin_rev" H 9675 4025 60  0001 C CNN
+F 2 "yosino46:SK6812MINI_rev" H 9675 4025 60  0001 C CNN
 F 3 "" H 9675 4025 60  0001 C CNN
 	1    9675 4025
@@
 F 0 "L5" H 9175 4287 51  0000 C CNN
 F 1 "SK6812MINI" H 9175 4222 16  0000 C CNN
-F 2 "yosino46:SK6812MINI_padin_rev" H 9175 4025 60  0001 C CNN
+F 2 "yosino46:SK6812MINI_rev" H 9175 4025 60  0001 C CNN
 F 3 "" H 9175 4025 60  0001 C CNN
 	1    9175 4025
@@
 F 0 "L4" H 8675 4287 51  0000 C CNN
 F 1 "SK6812MINI" H 8675 4222 16  0000 C CNN
-F 2 "yosino46:SK6812MINI_padin_rev" H 8675 4025 60  0001 C CNN
+F 2 "yosino46:SK6812MINI_rev" H 8675 4025 60  0001 C CNN
 F 3 "" H 8675 4025 60  0001 C CNN
 	1    8675 4025
@@
 F 0 "L3" H 8175 4287 51  0000 C CNN
 F 1 "SK6812MINI" H 8175 4222 16  0000 C CNN
-F 2 "yosino46:SK6812MINI_padin_rev" H 8175 4025 60  0001 C CNN
+F 2 "yosino46:SK6812MINI_rev" H 8175 4025 60  0001 C CNN
 F 3 "" H 8175 4025 60  0001 C CNN
 	1    8175 4025
@@
 F 0 "L2" H 7675 4287 51  0000 C CNN
 F 1 "SK6812MINI" H 7675 4222 16  0000 C CNN
-F 2 "yosino46:SK6812MINI_padin_rev" H 7675 4025 60  0001 C CNN
+F 2 "yosino46:SK6812MINI_rev" H 7675 4025 60  0001 C CNN
 F 3 "" H 7675 4025 60  0001 C CNN
 	1    7675 4025
@@
 F 0 "L1" H 7175 4287 51  0000 C CNN
 F 1 "SK6812MINI" H 7175 4222 16  0000 C CNN
-F 2 "yosino46:SK6812MINI_padin_rev" H 7175 4025 60  0001 C CNN
+F 2 "yosino46:SK6812MINI_rev" H 7175 4025 60  0001 C CNN
 F 3 "" H 7175 4025 60  0001 C CNN
 	1    7175 4025
@@
 F 0 "L7" H 7175 4313 51  0000 C CNN
 F 1 "SK6812MINI" H 7175 4378 16  0000 C CNN
-F 2 "yosino46:SK6812MINI_padin_rev" H 7175 4575 60  0001 C CNN
+F 2 "yosino46:SK6812MINI_rev" H 7175 4575 60  0001 C CNN
 F 3 "" H 7175 4575 60  0001 C CNN
 	1    7175 4575
@@
 F 0 "L8" H 7675 4313 51  0000 C CNN
 F 1 "SK6812MINI" H 7675 4378 16  0000 C CNN
-F 2 "yosino46:SK6812MINI_padin_rev" H 7675 4575 60  0001 C CNN
+F 2 "yosino46:SK6812MINI_rev" H 7675 4575 60  0001 C CNN
 F 3 "" H 7675 4575 60  0001 C CNN
 	1    7675 4575
@@
 F 0 "L9" H 8175 4313 51  0000 C CNN
 F 1 "SK6812MINI" H 8175 4378 16  0000 C CNN
-F 2 "yosino46:SK6812MINI_padin_rev" H 8175 4575 60  0001 C CNN
+F 2 "yosino46:SK6812MINI_rev" H 8175 4575 60  0001 C CNN
 F 3 "" H 8175 4575 60  0001 C CNN
 	1    8175 4575
@@
 F 0 "L10" H 8675 4313 51  0000 C CNN
 F 1 "SK6812MINI" H 8675 4378 16  0000 C CNN
-F 2 "yosino46:SK6812MINI_padin_rev" H 8675 4575 60  0001 C CNN
+F 2 "yosino46:SK6812MINI_rev" H 8675 4575 60  0001 C CNN
 F 3 "" H 8675 4575 60  0001 C CNN
 	1    8675 4575
@@
 F 0 "L11" H 9175 4313 51  0000 C CNN
 F 1 "SK6812MINI" H 9175 4378 16  0000 C CNN
-F 2 "yosino46:SK6812MINI_padin_rev" H 9175 4575 60  0001 C CNN
+F 2 "yosino46:SK6812MINI_rev" H 9175 4575 60  0001 C CNN
 F 3 "" H 9175 4575 60  0001 C CNN
 	1    9175 4575
@@
 F 0 "L12" H 9675 4313 51  0000 C CNN
 F 1 "SK6812MINI" H 9675 4378 16  0000 C CNN
-F 2 "yosino46:SK6812MINI_padin_rev" H 9675 4575 60  0001 C CNN
+F 2 "yosino46:SK6812MINI_rev" H 9675 4575 60  0001 C CNN
 F 3 "" H 9675 4575 60  0001 C CNN
 	1    9675 4575
@@
 F 0 "L18" H 9675 5387 51  0000 C CNN
 F 1 "SK6812MINI" H 9675 5322 16  0000 C CNN
-F 2 "yosino46:SK6812MINI_padin_rev" H 9675 5125 60  0001 C CNN
+F 2 "yosino46:SK6812MINI_rev" H 9675 5125 60  0001 C CNN
 F 3 "" H 9675 5125 60  0001 C CNN
 	1    9675 5125
@@
 F 0 "L17" H 9175 5387 51  0000 C CNN
 F 1 "SK6812MINI" H 9175 5322 16  0000 C CNN
-F 2 "yosino46:SK6812MINI_padin_rev" H 9175 5125 60  0001 C CNN
+F 2 "yosino46:SK6812MINI_rev" H 9175 5125 60  0001 C CNN
 F 3 "" H 9175 5125 60  0001 C CNN
 	1    9175 5125
@@
 F 0 "L16" H 8675 5387 51  0000 C CNN
 F 1 "SK6812MINI" H 8675 5322 16  0000 C CNN
-F 2 "yosino46:SK6812MINI_padin_rev" H 8675 5125 60  0001 C CNN
+F 2 "yosino46:SK6812MINI_rev" H 8675 5125 60  0001 C CNN
 F 3 "" H 8675 5125 60  0001 C CNN
 	1    8675 5125
@@
 F 0 "L15" H 8175 5387 51  0000 C CNN
 F 1 "SK6812MINI" H 8175 5322 16  0000 C CNN
-F 2 "yosino46:SK6812MINI_padin_rev" H 8175 5125 60  0001 C CNN
+F 2 "yosino46:SK6812MINI_rev" H 8175 5125 60  0001 C CNN
 F 3 "" H 8175 5125 60  0001 C CNN
 	1    8175 5125
@@
 F 0 "L14" H 7675 5387 51  0000 C CNN
 F 1 "SK6812MINI" H 7675 5322 16  0000 C CNN
-F 2 "yosino46:SK6812MINI_padin_rev" H 7675 5125 60  0001 C CNN
+F 2 "yosino46:SK6812MINI_rev" H 7675 5125 60  0001 C CNN
 F 3 "" H 7675 5125 60  0001 C CNN
 	1    7675 5125
@@
 F 0 "L13" H 7175 5387 51  0000 C CNN
 F 1 "SK6812MINI" H 7175 5322 16  0000 C CNN
-F 2 "yosino46:SK6812MINI_padin_rev" H 7175 5125 60  0001 C CNN
+F 2 "yosino46:SK6812MINI_rev" H 7175 5125 60  0001 C CNN
 F 3 "" H 7175 5125 60  0001 C CNN
 	1    7175 5125
@@
 F 0 "L19" H 7175 5413 51  0000 C CNN
 F 1 "SK6812MINI" H 7175 5478 16  0000 C CNN
-F 2 "yosino46:SK6812MINI_padin_rev" H 7175 5675 60  0001 C CNN
+F 2 "yosino46:SK6812MINI_rev" H 7175 5675 60  0001 C CNN
 F 3 "" H 7175 5675 60  0001 C CNN
 	1    7175 5675
@@
 F 0 "L20" H 7675 5413 51  0000 C CNN
 F 1 "SK6812MINI" H 7675 5478 16  0000 C CNN
-F 2 "yosino46:SK6812MINI_padin_rev" H 7675 5675 60  0001 C CNN
+F 2 "yosino46:SK6812MINI_rev" H 7675 5675 60  0001 C CNN
 F 3 "" H 7675 5675 60  0001 C CNN
 	1    7675 5675
@@
 F 0 "L21" H 8175 5413 51  0000 C CNN
 F 1 "SK6812MINI" H 8175 5478 16  0000 C CNN
-F 2 "yosino46:SK6812MINI_padin_rev" H 8175 5675 60  0001 C CNN
+F 2 "yosino46:SK6812MINI_rev" H 8175 5675 60  0001 C CNN
 F 3 "" H 8175 5675 60  0001 C CNN
 	1    8175 5675
@@
 F 0 "L22" H 8675 5413 51  0000 C CNN
 F 1 "SK6812MINI" H 8675 5478 16  0000 C CNN
-F 2 "yosino46:SK6812MINI_padin_rev" H 8675 5675 60  0001 C CNN
+F 2 "yosino46:SK6812MINI_rev" H 8675 5675 60  0001 C CNN
 F 3 "" H 8675 5675 60  0001 C CNN
 	1    8675 5675
@@
 F 0 "L23" H 9175 5413 51  0000 C CNN
 F 1 "SK6812MINI" H 9175 5478 16  0000 C CNN
-F 2 "yosino46:SK6812MINI_padin_rev" H 9175 5675 60  0001 C CNN
+F 2 "yosino46:SK6812MINI_rev" H 9175 5675 60  0001 C CNN
 F 3 "" H 9175 5675 60  0001 C CNN
 	1    9175 5675
